Commit message: adding flag to optionally add tactile sensors in xacro. default is true

File: barrett_hand_description/urdf/bh280.urdf.xacro (robot description, xacro)
@@ -12,5 +12,5 @@
 	<xacro:property name="joint_velocity_limit" value="2.0" />
 	<xacro:property name="mechanical_reduction" value="1.0" />
-	<xacro:macro name="bhand_macro" params="parent name *origin">
+	<xacro:macro name="bhand_macro" params="parent name *origin use_tactile_sensors:=true">
 		<joint name="${name}_base_joint" type="fixed">
 			<insert_block name="origin"/>
@@ -407,5 +407,7 @@
 		<link name="${name}_finger_34_link"/>
 		<!-- Auto generated tactile sensor links -->
-		<xacro:bh_tactile name="bh"/>
+		<xacro:if value="${use_tactile_sensors}">
+			<xacro:bh_tactile name="bh"/>
+		</xacro:if>
 	</xacro:macro>
 </robot>
